File: docs/03-build/04-pcbs/pcb-15-nose-hall/design/pcb-15-nose-hall.kicad_sch (KiCad schematic)
At the start: 7 parts, among them P1 +3V3 wire, P2 GND wire, P3 HALL_OUT wire, U1 DRV5055A3QDBZR

Commit message: build(pcbs): PCB-15 nose Hall carrier rev A; board moved 0.4 mm back (D-061..D-063)
PCB-15 completes stage 1 (design) of the 04-pcbs workflow:
- Schematic (ERC 0/0) and a hand-routed 2-layer layout through KiPy on the
  KiCad 10.99 nightly: U1 on the front with three via fan-outs, C1/C2/R1 and
  the wire pads on the back. DRC with schematic parity: 0 errors.
- Custom U1 land pattern SOT-23_NoseNotch (toes trimmed to fit the seat notch).
- Fab-neutral rules for JLCPCB, PCBWay and Lion Circuits MII (D-061, D-062)
  in design/pcb-15-nose-hall.kicad_dru; the board is laid out to them.
- Rev A outputs in fab/revA/ (Gerber X2, Excellon, placement, BOM, zip,
  order notes) and the board STEP in cad/.

The stage-1 fit check (final/v1/cad/check_pcb15_fit.py) found that the
magnet could hit U1 at the cap's 3 mm stop (-0.205 mm worst case). D-063
moves the board and its 1.0 mm slot 0.4 mm back and deepens the D-059
relief to 1.3 mm, all in final/v1/cad via new DROID_ADDS and DROID_MOVES
tables. Fit and relief checks pass (worst-case air +0.195 mm); both droid
STEPs rebuilt. Predicted trip moves from 0.73 to 0.89 mm of travel.

Also ignores KiCad's .history/ local-history folders.

Co-Authored-By: Claude Opus 5.5 <noreply@anthropic.com>
Parts:
- U1: footprint Package_TO_SOT_SMD:SOT-23 -> pcb15:SOT-23_NoseNotch
