File: docs/03-build/04-pcbs/pcb-10-c3-carrier/design/pcb-10-c3-carrier.kicad_sch (KiCad schematic)
At the start: 90 parts, among them J1 J10-1 +5 V (W11), J10 J10-10 rear TCRT (W36), J12 J10-12 readiness (W39, PCB-03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, J2 J10-2 base link (W25), J3 J10-3 encoder L (W30), J4 J10-4 encoder R (W31), J5 J10-5 left DRV8833 (W32), J6 J10-6 right DRV8833 (W33), J7 J10-7 IMU PCB-07 (W29), J8 J10-8 nose (W34), Q1 AO3400A, U1 ESP32-S3-DevKitC-1-N8, U2 THVD1451DR, U3 TPS3436CCCBGDDFRQ1, U4 74LVC1G08, U5 74LVC1G11

Commit message: build(pcbs): PCB-10 board set-up; third connector row, notched outline, 3D models (D-068 amended, lesson 3)
The real connector footprints at the CAD positions gave 23 courtyard
overlaps on a scratch board: GH rows 6 mm apart against 6.6 mm courtyards,
and the real Micro-Fit (9.65 x 9.9 mm) over three GH headers. The board
grows 6 mm down (70 x 49.5) for a third row, notched over the right
DRV8833's terminal block; J10-1 keeps its RA Micro-Fit at the real size.
Final CAD follows; check_pcb10_mount.py 9/9 pass.

Board file: outline, 1.6 mm stackup, origins, B-side rule areas over the
uprights and F-side ones under the hooks (proved on a scratch copy with
its own rules), placement drawings. Empty-board DRC 0 violations.
3D models: TSOT-23-8 for the DDF watchdog (checked against TI 4222047/E),
full-tail Micro-Fit from Molex SD-43650-001; both land on their pads.

Co-Authored-By: Claude Opus 5.5 <noreply@anthropic.com>
Parts:
- J1: footprint Connector_Molex:Molex_Micro-Fit_3.0_43650-0200_1x02_P3.00mm_Horizontal -> pcb10:Molex_Micro-Fit_3.0_43650-0200_1x02_P3.00mm_Horizontal
- U3: footprint Package_TO_SOT_SMD:Texas_DDF0008A_SOT-8_1.6x2.9mm_P0.65mm -> pcb10:Texas_DDF0008A_SOT-8_1.6x2.9mm_P0.65mm

Commit message: build(pcbs): PCB-10 placement, DRC clean; J10-2 reordered, GPIO map v0.3 for routing (lesson 4, part 1)
All 90 footprints placed through KiPy on the proved connector origins;
DRC: no courtyard, edge or parity errors (53 cosmetic rotated-footprint
library mismatches, the PCB-15 trap). J10-2 takes U2's own pin order so
the RS-422 pairs run straight (PCB-09 and 05-harness updated); the GPIO
map is reassigned (v0.3) so each pin sits next to the connector it feeds.
Schematic regenerated, ERC 0/0, board pad nets updated to match.

Co-Authored-By: Claude Opus 5.5 <noreply@anthropic.com>
Connections:
- net C0TX_N: now also J2.3 (Pin_3); no longer J2.5 (Pin_5)
- net C0TX_P: now also J2.2 (Pin_2); no longer J2.4 (Pin_4)
- net C3TX_N: now also J2.4 (Pin_4); no longer J2.3 (Pin_3)
- net C3TX_P: now also J2.5 (Pin_5); no longer J2.2 (Pin_2)
- net ENC_L_A: now also U1.8 (GPIO15/ADC2_CH4/32K_P); no longer U1.4 (GPIO4/ADC1_CH3)
- net ENC_L_B: now also U1.9 (GPIO16/ADC2_CH5/32K_N); no longer U1.5 (GPIO5/ADC1_CH4)
- net HALL_ADC: now also U1.40 (GPIO2/ADC1_CH1); no longer U1.16 (GPIO10/ADC1_CH9)
- net IMU_CS_MCU: now also U1.17 (GPIO11/ADC2_CH0); no longer U1.38 (GPIO41/MTDI)
- net IMU_INT1_MCU: now also U1.18 (GPIO12/ADC2_CH1); no longer U1.39 (GPIO42/MTMS)
- net IMU_MISO_MCU: now also U1.16 (GPIO10/ADC1_CH9); no longer U1.33 (GPIO36)
- net IMU_MOSI_MCU: now also U1.15 (GPIO9/ADC1_CH8); no longer U1.32 (GPIO35)
- net IMU_SCLK_MCU: now also U1.12 (GPIO8/ADC1_CH7); no longer U1.34 (GPIO37)
- net IN1_L_MCU: now also U1.34 (GPIO37); no longer U1.17 (GPIO11/ADC2_CH0)
- net IN1_R_MCU: now also U1.39 (GPIO42/MTMS); no longer U1.18 (GPIO12/ADC2_CH1)
- net IN2_L_MCU: now also U1.33 (GPIO36); no longer U1.19 (GPIO13/ADC2_CH2)
- net IN2_R_MCU: now also U1.38 (GPIO41/MTDI); no longer U1.20 (GPIO14/ADC2_CH3)
- net MCU_RDY: now also U1.28 (GPIO47); no longer U1.40 (GPIO2/ADC1_CH1)
- net MOTOR_PRESENT_MCU: now also U1.10 (GPIO17/ADC2_CH6); no longer U1.37 (GPIO40/MTDO)
- net NFAULT: now also U1.11 (GPIO18/ADC2_CH7); no longer U1.15 (GPIO9/ADC1_CH8)
- net TCRT_ADC: now also U1.5 (GPIO5/ADC1_CH4); no longer U1.12 (GPIO8/ADC1_CH7)
- net TCRT_LED_EN: now also U1.4 (GPIO4/ADC1_CH3); no longer U1.28 (GPIO47)
- net UART_RX: now also U1.19 (GPIO13/ADC2_CH2); no longer U1.11 (GPIO18/ADC2_CH7)
- net UART_TX: now also U1.20 (GPIO14/ADC2_CH3); no longer U1.10 (GPIO17/ADC2_CH6)
Other:
- note added: "GPIO map v0.3 (layout): pins chosen so each track runs to its connector without crossings. Unused: GPIO0/3/45/46 (strapping), 19/20/43/44 (USB), 35/39/40 (spares), 38 (v1.1 RGB LED)."
- note added: "J10-2 (D-068 F, reordered at placement): 1 GND, 2/3 C0TX+/- (U2 A/B, 120R here), 4/5 C3TX-/+ (U2 Z/Y), 6 spare: U2's own pin order, so the pairs run straight. W25 1:1; PCB-09 J9-2 mirrors it."
- note removed: "J10-2 (D-068 F): 1 GND, 2/3 C3TX+/- (U2 Y/Z), 4/5 C0TX+/- (U2 A/B, 120R here), 6 spare. W25 1:1; PCB-09 J9-2 mirrors it."
- note removed: "Unused: GPIO0/3/45/46 (strapping), 19/20/43/44 (USB), 15/16/39 (spares), 38 (v1.1 RGB LED)."
