File: project/03-build/04-pcbs/pcb-13-charge-inlet/design/pcb-13-charge-inlet.kicad_sch (KiCad schematic)
At the start: 30 parts, among them J1 USB4140-GF-0170-C, J2 W16 pads, Q1 STL6P3LLH6, U1 STUSB4500QTR

Commit message: build(pcbs): PCB-13 placed and routed (lesson 4); DRC 0 errors, 0 unconnected, parity clean
Hand-routed, octolinear, two layers at 1 oz. 3 A path as pours: VBUS 2.41 mm narrowest,
VSNK 1.29 mm past H2. D-069 amended at placement: ADDR0/ADDR1/RESET to GND (R5-R7 out),
TP5-TP8 out, D2 inputs swapped, J2 turned 180. New playbook traps: KiPy is_rule_area()
is a method; plan a crowded QFN's orientation first.

Co-Authored-By: Claude Opus 5.5 <noreply@anthropic.com>
Parts:
- removed R5, R6, R7: 100k, Resistor_SMD:R_0402_1005Metric, symbol Device:R
- removed TP5: RESET, TestPoint:TestPoint_Pad_D1.0mm, symbol Connector:TestPoint
- removed TP6: VSNK, TestPoint:TestPoint_Pad_D1.0mm, symbol Connector:TestPoint
- removed TP7: CC1, TestPoint:TestPoint_Pad_D1.0mm, symbol Connector:TestPoint
- removed TP8: CC2, TestPoint:TestPoint_Pad_D1.0mm, symbol Connector:TestPoint
Connections:
- net ADDR0 is gone; now on net GND: U1.12 (ADDR0)
- net ADDR1 is gone; now on net GND: U1.13 (ADDR1)
- net RESET is gone; now on net GND: U1.6 (RESET)
- net CC1: now also D2.2 (K); no longer D2.1 (K)
- net CC2: now also D2.1 (K); no longer D2.2 (K)
Other:
- note added: "PCB-13 charge inlet, rev A. Spec: charge-path.md sec 3 (D-040), inputs frozen in D-069 (04-pcbs/pcb-13-charge-inlet/README.md). J1 GCT USB4140-GF-0170-C on the -X (panel) face, hand-soldered by the builder (D-069): VBUS A9/B9, GND A12/B12 and the four shell stakes (SH), CC1 A5, CC2 B5. D1 TVS2200 (22 V stand-off, 28.35 V max clamp) and C1 at J1; D2 ESDA25W on CC1 (pin 2) and CC2 (pin 1): identica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"
- note removed: "PCB-13 charge inlet, rev A. Spec: charge-path.md sec 3 (D-040), inputs frozen in D-069 (04-pcbs/pcb-13-charge-inlet/README.md). J1 GCT USB4140-GF-0170-C on the -X (panel) face, hand-soldered by the builder (D-069): VBUS A9/B9, GND A12/B12 and the four shell stakes (SH), CC1 A5, CC2 B5. D1 TVS2200 (22 V stand-off, 28.35 V max clamp) and C1 at J1; D2 ESDA25W on CC1/CC2. Everything on VBUS is rated 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"
- moved on the sheet: TP10, TP9
